File: cosel_dc-dc_board/cosel_dc-dc_board.kicad_pcb (KiCad board)
At the start: 2 copper layers, 110 x 80 mm, 11 parts, among them J1 B2PS-VH(LF)(SN), J2 B2PS-VH(LF)(SN), J3 S3B-XH-A(LF)(SN), U1 CBS

Commit message: update
Parts:
- added D1: LED, LED_SMD:LED_0603_1608Metric_Pad1.05x0.95mm_HandSolder, F.Cu at (25.4, 72.4)
- added D2: LED, LED_SMD:LED_0603_1608Metric_Pad1.05x0.95mm_HandSolder, F.Cu at (86.4, 72.4)
- added R1: 10k, Resistor_SMD:R_0603_1608Metric_Pad1.05x0.95mm_HandSolder, F.Cu at (29.2, 72.4)
- added R2: 10k, Resistor_SMD:R_0603_1608Metric_Pad1.05x0.95mm_HandSolder, F.Cu at (82.5, 72.4)
Routing:
- net GND: track 66.4 -> 134.2 mm
- net +24V: track 50.6 -> 71.5 mm
- net Net-(C2-Pad1): track 56.9 -> 69.6 mm
- net Net-(D2-Pad1): track 0.00 -> 2.06 mm
- net Net-(D1-Pad1): track 0.00 -> 2.06 mm
Other:
- board text added: "COSEL CBS Series DC-DC Converter Board"
- board text removed: "COSEL CBS Series DC-DC converter board"

Commit message: update
Parts:
- removed J3: S3B-XH-A(LF)(SN), SamacSys_Parts:SHDR3W80P0X250_1X3_990X610X700P
- J2: value B2PS-VH(LF)(SN) -> Screw_Terminal_01x02; footprint SamacSys_Parts:B2PS-VH -> TerminalBlock:TerminalBlock_Altech_AK300-2_P5.00mm
- moved REF** 5.00 mm to (100.0, 75.0)
- moved REF** 5.00 mm to (100.0, 5.00)
- moved J2 3.47 mm to (95.0, 61.5)
Connections:
- J2 pad 1: Net-(C2-Pad1) -> Net-(C2-Pad2)
- J2 pad 2: Net-(C2-Pad2) -> Net-(C2-Pad1)
Routing:
- net Net-(C2-Pad2): track 62.9 -> 69.9 mm
- net Net-(C2-Pad1): track 69.6 -> 74.0 mm
- removed copper zone on B.Cu, net GND
- removed copper zone on F.Cu, net GND
Other:
- board size 110 x 80 mm -> 105 x 80 mm

Commit message: update
Parts:
- added J3: Screw_Terminal_01x02, TerminalBlock:TerminalBlock_bornier-2_P5.08mm, F.Cu at (10.2, 62.2)
- J2: footprint TerminalBlock:TerminalBlock_Altech_AK300-2_P5.00mm -> TerminalBlock:TerminalBlock_bornier-2_P5.08mm
- moved J2 86.0 mm to (10.0, 48.3), turned to 270 degrees
- moved C2 81.6 mm to (8.64, 27.9)
- moved C1 79.7 mm to (90.7, 58.0)
- moved J1 75.8 mm to (90.4, 31.2), turned to 90 degrees
- moved LED2 55.0 mm to (31.4, 72.4)
- moved R2 55.0 mm to (27.6, 72.4)
- moved LED1 51.4 mm to (76.8, 72.5)
- moved R1 51.4 mm to (80.6, 72.5)
- moved U1 0.58 mm to (54.4, 38.1), turned to 180 degrees
- renumbered D1 to LED1, D2 to LED2
Connections:
- C2 pad 2: Net-(C2-Pad2) -> GNDPWR
- J2 pad 1: Net-(C2-Pad2) -> GNDPWR
- R2 pad 2: GND -> GNDPWR
- U1 pad 5: Net-(C2-Pad2) -> Net-(C2-Pad1)
- U1 pad 6: Net-(C2-Pad2) -> Net-(C2-Pad1)
- U1 pad 8: Net-(C2-Pad1) -> GNDPWR
- U1 pad 9: Net-(C2-Pad1) -> GNDPWR
Routing:
- net GNDPWR: track 0.00 -> 101.5 mm
- net Net-(C2-Pad2): track 69.9 -> 0.00 mm
- net GND: track 134.2 -> 77.4 mm
- net Net-(C2-Pad1): track 74.0 -> 94.4 mm
- net +24V: track 71.5 -> 60.4 mm
- added copper zone on F.Cu, net GND
- added copper zone on B.Cu, net GNDPWR

Commit message: update
Parts:
- moved J1 6.60 mm to (83.8, 31.2)
- moved REF** 5.00 mm to (95.0, 75.0)
- moved REF** 5.00 mm to (95.0, 5.00)
- moved C1 4.32 mm to (86.4, 58.0)
- moved U1 2.62 mm to (52.1, 36.8)
- moved R2 2.54 mm to (25.0, 72.4)
- moved LED2 2.54 mm to (28.8, 72.4)
- moved LED1 1.27 mm to (75.6, 72.5)
- moved R1 1.27 mm to (79.4, 72.5)
Routing:
- net GNDPWR: track 101.5 -> 143.2 mm
- net GND: track 77.4 -> 71.3 mm
- net Net-(C2-Pad1): track 94.4 -> 99.8 mm
- net +24V: track 60.4 -> 59.0 mm
- added copper zone on B.Cu, net GND
- added copper zone on F.Cu, net GNDPWR
- removed copper zone on F.Cu, net GND
- removed copper zone on B.Cu, net GNDPWR
Other:
- board size 105 x 80 mm -> 100 x 80 mm

Commit message: update
Parts:
- J1: value B2PS-VH(LF)(SN) -> Conn_01x02; footprint SamacSys_Parts:B2PS-VH -> Connector_JST:JST_VH_S2P-VH_1x02_P3.96mm_Horizontal
- moved J1 2.18 mm to (85.1, 33.0)
Routing:
- net GND: track 71.3 -> 82.4 mm
- net +24V: track 59.0 -> 60.4 mm

Commit message: update
Parts:
- C1: footprint Capacitor_THT:CP_Radial_D16.0mm_P7.50mm -> Capacitor_THT:CP_Radial_D6.3mm_P2.50mm
- moved C1 8.60 mm to (87.6, 49.5), turned to 180 degrees
Routing:
- net GNDPWR: track 143.2 -> 107.3 mm
- net GND: track 82.4 -> 74.9 mm
- net +24V: track 60.4 -> 64.8 mm
- removed copper zone on B.Cu, net GND
