File: power_control_board/power_control_board.kicad_pcb (KiCad board)
At the start: 2 copper layers, 80 x 50 mm, 14 parts, among them J1 B2PS-VH(LF)(SN), J2 S3B-XH-A(LF)(SN), J3 B2PS-VH(LF)(SN), Q1 2SC2712-Y(F)

Commit message: update
Parts:
- removed Q1: 2SC2712-Y(F), SC-59
- added J4: Conn_01x02, Connector_JST:JST_XH_S2B-XH-A-1_1x02_P2.50mm_Horizontal, F.Cu at (124.5, 87.6)
- added LED1: LED, LED_SMD:LED_0603_1608Metric_Pad1.05x0.95mm_HandSolder, F.Cu at (100.3, 54.6)
- added R3: 1k, Resistor_SMD:R_0603_1608Metric_Pad1.05x0.95mm_HandSolder, F.Cu at (96.5, 54.6)
- J1, J3: value B2PS-VH(LF)(SN) -> Conn_01x02; footprint SamacSys_Parts:B2PS-VH -> Connector_JST:JST_VH_B2PS-VH_1x02_P3.96mm_Horizontal
- J2: value S3B-XH-A(LF)(SN) -> Conn_01x03; footprint SamacSys_Parts:SHDR3W80P0X250_1X3_990X610X700P -> Connector_JST:JST_XH_S3B-XH-A-1_1x03_P2.50mm_Horizontal
- R1: footprint Resistor_THT:R_Axial_DIN0309_L9.0mm_D3.2mm_P12.70mm_Horizontal -> Resistor_SMD:R_0603_1608Metric_Pad1.05x0.95mm_HandSolder
- R2: value 1k -> 2k; footprint Resistor_THT:R_Axial_DIN0309_L9.0mm_D3.2mm_P12.70mm_Horizontal -> Resistor_SMD:R_0603_1608Metric_Pad1.05x0.95mm_HandSolder
- moved R2 55.9 mm to (125.7, 92.7), turned to 180 degrees
- moved R1 24.3 mm to (121.9, 92.7)
- moved J2 10.5 mm to (69.8, 77.5), turned to 270 degrees
- moved C1 7.62 mm to (120.7, 61.0)
- moved J1 6.07 mm to (121.9, 78.7)
- moved J3 1.80 mm to (77.5, 64.8)
- renumbered RELAY to K1
Connections:
- D1 pad 2: Net-(D1-Pad2) -> GNDD
- J2 pad 1: +5V -> GNDD
- J2 pad 3: GNDD -> +5V
- K1 pad 2: Net-(D1-Pad2) -> GNDD
- R1 pad 1: GNDD -> Net-(J4-Pad2)
- R1 pad 2: Net-(Q1-Pad1) -> +5V
- R2 pad 1: +5V -> GNDD
- R2 pad 2: Net-(Q1-Pad1) -> Net-(J4-Pad2)
Routing:
- net GNDD: track 35.7 -> 67.4 mm
- net Net-(D1-Pad2): track 19.6 -> 0.00 mm
- net Net-(C1-Pad1): track 26.9 -> 45.3 mm
- net GND: track 80.8 -> 93.8 mm
- net Net-(J4-Pad2): track 0.00 -> 11.1 mm
- net Net-(Q1-Pad1): track 10.7 -> 0.00 mm
- net +5V: track 63.4 -> 70.0 mm
- net Net-(LED1-Pad1): track 0.00 -> 2.06 mm
- net +24V: track 16.3 -> 14.7 mm
Other:
- board text added: "3.3V output"

Commit message: update
Parts:
- D1: footprint SamacSys_Parts:DIOAD1340W57L300D260 -> Diode_THT:D_DO-41_SOD81_P7.62mm_Horizontal
- moved D1 28.2 mm to (101.6, 93.1), turned to 180 degrees
Routing:
- net +5V: track 70.0 -> 81.6 mm
- net GNDD: track 67.4 -> 75.3 mm
- net Net-(J4-Pad2): track 11.1 -> 12.9 mm
- added copper zone on B.Cu, net GND
- removed copper zone on B.Cu, net GNDD
